Commit message: astrid_slam

File: astrid_description/urdf/astrid.urdf.xacro (robot description, xacro)
@@ -133,43 +133,4 @@
     <!-- <fdir1 value="1 0 0"/> -->
   </xacro:macro>
-  <!-- Battery
-  <xacro:macro name="battery" params="prefix reflect">
-    <joint name="chassis_to_${prefix}_battery" type="fixed">
-      <parent link="chassis" />
-      <child link="${prefix}_battery_offset" />
-      <origin xyz="${battery_x_offset - battery_length / 2}
-                   ${reflect * battery_dist / 2}
-                   0" rpy="${reflect * battery_comp_angle} 0 0" />
-    </joint>
-    <link name="${prefix}_battery_offset">
-      <xacro:null_inertial />
-    </link>
-    <joint name="offset_to_${prefix}_battery" type="fixed">
-      <parent link="${prefix}_battery_offset" />
-      <child link="${prefix}_battery" />
-      <origin xyz="0
-                   ${reflect * battery_width / 2}
-                   ${(battery_height / 2) - battery_comp_depth}" />
-    </joint>
-    <link name="${prefix}_battery">
-      <visual>
-        <geometry>
-          <box size="${battery_length} ${battery_width} ${battery_height}" />
-        </geometry>
-        <material name="battery_mat" />
-      </visual>
-      <collision>
-        <geometry>
-          <box size="${battery_length} ${battery_width} ${battery_height}" />
-        </geometry>
-      </collision>
-      <xacro:solid_cuboid_inertial width="${battery_length}" depth="${battery_width}" height="${battery_height}" mass="${battery_mass}">
-        <origin />
-      </xacro:solid_cuboid_inertial>
-    </link>
-    <gazebo reference="${prefix}_battery">
-      <material>Gazebo/Blue</material>
-    </gazebo>
-  </xacro:macro> -->
   <!-- Shock absorber -->
   <xacro:macro name="shock" params="lr_prefix fr_prefix lr_reflect fr_reflect child">
@@ -282,15 +243,5 @@
   <!-- base_link must have geometry so that its axes can be displayed in
        rviz. -->
-  <link name="base_link">
-    <visual>
-      <geometry>
-        <box size="0.01 0.01 0.01" />
-      </geometry>
-      <material name="chassis_mat" />
-    </visual>
-  </link>
-  <gazebo reference="base_link">
-    <material>Gazebo/Grey</material>
-  </gazebo>
+  <link name="base_link" />
   <!-- Chassis -->
   <link name="chassis">
@@ -429,5 +380,5 @@
 </xacro:macro>
   <joint name="laser_base_joint" type="fixed">
-    <origin xyz="1.005 -0.032 0.41" rpy="0 0.0 0.0" />
+    <origin xyz="1.2 -0.032 0.3" rpy="0 0.0 0.0" />
     <!-- <origin xyz = "0 0 0.025" rpy="0 0 -1.57"/> -->
     <parent link="chassis" />
@@ -452,12 +403,12 @@
       <pose>0 0 0 0 0 0</pose>
       <visualize>true</visualize>
-      <update_rate>40</update_rate>
+      <update_rate>50</update_rate>
       <ray>
         <scan>
           <horizontal>
-            <samples>720</samples>
+            <samples>360</samples>
             <resolution>1</resolution>
-            <min_angle>-1.57</min_angle>
-            <max_angle>1.57</max_angle>
+            <min_angle>-1.57079</min_angle>
+            <max_angle>1.57079</max_angle>
           </horizontal>
         </scan>

Commit message: updated slam and added navigation

File: astrid_description/urdf/astrid.urdf.xacro (robot description, xacro)
@@ -122,5 +122,5 @@
     <mu1 value="1.0"/>
     <mu2 value="1.0"/>
-    <kp  value="10000000.0" />
+    <kp  value="15000000.0" />
     <kd  value="1.0" />
     <fdir1 value="1 0 0"/>
@@ -331,5 +331,5 @@
   <gazebo reference="camera_link">
     <sensor type="camera" name="main_camera">
-      <update_rate>30.0</update_rate>
+      <!-- <update_rate>30.0</update_rate> -->
       <camera name="head">
         <horizontal_fov>1.3962634</horizontal_fov>
@@ -354,6 +354,6 @@
       <plugin name="camera_controller" filename="libgazebo_ros_camera.so">
         <alwaysOn>true</alwaysOn>
-        <updateRate>0.0</updateRate>
-        <cameraName>astrid/camera</cameraName>
+        <updateRate>30.0</updateRate>
+        <cameraName>camera</cameraName>
         <imageTopicName>image_raw</imageTopicName>
         <cameraInfoTopicName>camera_info</cameraInfoTopicName>
@@ -369,5 +369,5 @@
   </gazebo>
   <!-- laser -->
-<xacro:macro name="laser_base_geometry">
+<xacro:macro name="base_scan_geometry">
   <geometry>
     <cylinder length="0.05" radius="0.05" />
@@ -379,13 +379,13 @@
   </geometry>
 </xacro:macro>
-  <joint name="laser_base_joint" type="fixed">
+  <joint name="base_scan_joint" type="fixed">
     <origin xyz="1.2 -0.032 0.3" rpy="0 0.0 0.0" />
     <!-- <origin xyz = "0 0 0.025" rpy="0 0 -1.57"/> -->
     <parent link="chassis" />
-    <child link="laser_base" />
+    <child link="base_scan" />
   </joint>
-  <link name="laser_base">
+  <link name="base_scan">
       <visual>
-          <xacro:laser_base_geometry />
+          <xacro:base_scan_geometry />
       </visual>
       <inertial>
@@ -394,10 +394,10 @@
       </inertial>
   </link>
-  <gazebo reference="laser_base">
+  <gazebo reference="base_scan">
     <material>Gazebo/Grey</material>
     <mu1>0.2</mu1>
     <mu2>0.2</mu2>
   </gazebo>
-  <gazebo reference="laser_base">
+  <gazebo reference="base_scan">
     <sensor type="ray" name="lidar">
       <pose>0 0 0 0 0 0</pose>
@@ -407,5 +407,5 @@
         <scan>
           <horizontal>
-            <samples>360</samples>
+            <samples>720</samples>
             <resolution>1</resolution>
             <min_angle>-1.57079</min_angle>
@@ -415,5 +415,5 @@
         <range>
           <min>0.10</min>
-          <max>30.0</max>
+          <max>12.0</max>
           <resolution>0.01</resolution>
         </range>
@@ -430,12 +430,78 @@
       <plugin name="lidar_controller" filename="libgazebo_ros_laser.so">
         <!-- <robotNamespace>astrid</robotNamespace> -->
-        <topicName>astrid/scan</topicName>
-        <frameName>laser_base</frameName>
+        <topicName>scan</topicName>
+        <frameName>base_scan</frameName>
         <alwaysOn>true</alwaysOn>
       </plugin>
     </sensor>
   </gazebo>
+  <!-- Top View Camera-->
+  <joint name="top_view_camera_joint" type="fixed">
+    <axis xyz="0 1 0" />
+    <!-- <origin xyz="0 4.2 2.5" rpy="0 0.2 -1.57"/> -->
+    <origin xyz="-3 0 1.8" rpy="0 0 0" />
+    <parent link="shell"/>
+    <child link="top_view_camera_link"/>
+  </joint>
+  <link name="top_view_camera_link">
+    <visual>
+      <origin xyz="0 0 0" rpy="0 0 0"/>
+      <geometry>
+    <box size="0.05 0.07 0.03"/>
+      </geometry>
+      <material name="red"/>
+    </visual>
+    <inertial>
+      <mass value="1e-5" />
+      <origin xyz="0 0 0" rpy="0 0 0"/>
+      <inertia ixx="1e-6" ixy="0" ixz="0" iyy="1e-6" iyz="0" izz="1e-6" />
+    </inertial>
+  </link>
+<!-- top view camera -->
+    <gazebo reference="top_view_camera_link">
+      <sensor type="camera" name="top_view_camera">
+        <update_rate>30.0</update_rate>
+        <camera name="top_view_head">
+          <horizontal_fov>1.3962634</horizontal_fov>
+          <image>
+            <width>1600</width>
+            <height>900</height>
+            <format>R8G8B8</format>
+          </image>
+          <clip>
+            <near>0.02</near>
+            <far>500</far>
+          </clip>
+          <noise>
+            <type>gaussian</type>
+            <!-- Noise is sampled independently per pixel on each frame.
+                 That pixel's noise value is added to each of its color
+                 channels, which at that point lie in the range [0,1]. -->
+            <mean>0.0</mean>
+            <stddev>0.007</stddev>
+          </noise>
+        </camera>
+        <plugin name="camera_controller" filename="libgazebo_ros_camera.so">
+          <alwaysOn>true</alwaysOn>
+          <updateRate>0.0</updateRate>
+          <cameraName>astrid/top_view_camera</cameraName>
+          <imageTopicName>image_raw</imageTopicName>
+          <cameraInfoTopicName>camera_info</cameraInfoTopicName>
+          <frameName>camera_link</frameName>
+          <hackBaseline>0.07</hackBaseline>
+          <distortionK1>0.0</distortionK1>
+          <distortionK2>0.0</distortionK2>
+          <distortionK3>0.0</distortionK3>
+          <distortionT1>0.0</distortionT1>
+          <distortionT2>0.0</distortionT2>
+        </plugin>
+      </sensor>
+    </gazebo>
   <gazebo>
     <plugin name="gazebo_ros_control" filename="libgazebo_ros_control.so" />
+    <robotBaseFrame>base_link</robotBaseFrame>
+    <commandTopic>cmd_vel</commandTopic>
+      <odometryTopic>odom</odometryTopic>
+      <odometryFrame>odom</odometryFrame>
   </gazebo>
 </robot>

Commit message: navigation optimization done by mk

File: astrid_description/urdf/astrid.urdf.xacro (robot description, xacro)
@@ -122,5 +122,5 @@
     <mu1 value="1.0"/>
     <mu2 value="1.0"/>
-    <kp  value="10000000.0" />
+    <kp  value="15000000.0" />
     <kd  value="1.0" />
     <fdir1 value="1 0 0"/>
@@ -133,43 +133,4 @@
     <!-- <fdir1 value="1 0 0"/> -->
   </xacro:macro>
-  <!-- Battery
-  <xacro:macro name="battery" params="prefix reflect">
-    <joint name="chassis_to_${prefix}_battery" type="fixed">
-      <parent link="chassis" />
-      <child link="${prefix}_battery_offset" />
-      <origin xyz="${battery_x_offset - battery_length / 2}
-                   ${reflect * battery_dist / 2}
-                   0" rpy="${reflect * battery_comp_angle} 0 0" />
-    </joint>
-    <link name="${prefix}_battery_offset">
-      <xacro:null_inertial />
-    </link>
-    <joint name="offset_to_${prefix}_battery" type="fixed">
-      <parent link="${prefix}_battery_offset" />
-      <child link="${prefix}_battery" />
-      <origin xyz="0
-                   ${reflect * battery_width / 2}
-                   ${(battery_height / 2) - battery_comp_depth}" />
-    </joint>
-    <link name="${prefix}_battery">
-      <visual>
-        <geometry>
-          <box size="${battery_length} ${battery_width} ${battery_height}" />
-        </geometry>
-        <material name="battery_mat" />
-      </visual>
-      <collision>
-        <geometry>
-          <box size="${battery_length} ${battery_width} ${battery_height}" />
-        </geometry>
-      </collision>
-      <xacro:solid_cuboid_inertial width="${battery_length}" depth="${battery_width}" height="${battery_height}" mass="${battery_mass}">
-        <origin />
-      </xacro:solid_cuboid_inertial>
-    </link>
-    <gazebo reference="${prefix}_battery">
-      <material>Gazebo/Blue</material>
-    </gazebo>
-  </xacro:macro> -->
   <!-- Shock absorber -->
   <xacro:macro name="shock" params="lr_prefix fr_prefix lr_reflect fr_reflect child">
@@ -282,15 +243,5 @@
   <!-- base_link must have geometry so that its axes can be displayed in
        rviz. -->
-  <link name="base_link">
-    <visual>
-      <geometry>
-        <box size="0.01 0.01 0.01" />
-      </geometry>
-      <material name="chassis_mat" />
-    </visual>
-  </link>
-  <gazebo reference="base_link">
-    <material>Gazebo/Grey</material>
-  </gazebo>
+  <link name="base_link" />
   <!-- Chassis -->
   <link name="chassis">
@@ -380,10 +331,10 @@
   <gazebo reference="camera_link">
     <sensor type="camera" name="main_camera">
-      <update_rate>30.0</update_rate>
+      <!-- <update_rate>30.0</update_rate> -->
       <camera name="head">
         <horizontal_fov>1.3962634</horizontal_fov>
         <image>
-          <width>1600</width>
-          <height>900</height>
+          <width>1280</width>
+          <height>720</height>
           <format>R8G8B8</format>
         </image>
@@ -403,6 +354,6 @@
       <plugin name="camera_controller" filename="libgazebo_ros_camera.so">
         <alwaysOn>true</alwaysOn>
-        <updateRate>0.0</updateRate>
-        <cameraName>astrid/camera</cameraName>
+        <updateRate>10.0</updateRate>
+        <cameraName>camera</cameraName>
         <imageTopicName>image_raw</imageTopicName>
         <cameraInfoTopicName>camera_info</cameraInfoTopicName>
@@ -418,5 +369,5 @@
   </gazebo>
   <!-- laser -->
-<xacro:macro name="laser_base_geometry">
+<xacro:macro name="base_scan_geometry">
   <geometry>
     <cylinder length="0.05" radius="0.05" />
@@ -428,13 +379,13 @@
   </geometry>
 </xacro:macro>
-  <joint name="laser_base_joint" type="fixed">
-    <origin xyz="1.005 -0.032 0.41" rpy="0 0.0 0.0" />
+  <joint name="base_scan_joint" type="fixed">
+    <origin xyz="1.2 -0.032 0.3" rpy="0 0.0 0.0" />
     <!-- <origin xyz = "0 0 0.025" rpy="0 0 -1.57"/> -->
     <parent link="chassis" />
-    <child link="laser_base" />
+    <child link="base_scan" />
   </joint>
-  <link name="laser_base">
+  <link name="base_scan">
       <visual>
-          <xacro:laser_base_geometry />
+          <xacro:base_scan_geometry />
       </visual>
       <inertial>
@@ -443,14 +394,14 @@
       </inertial>
   </link>
-  <gazebo reference="laser_base">
+  <gazebo reference="base_scan">
     <material>Gazebo/Grey</material>
     <mu1>0.2</mu1>
     <mu2>0.2</mu2>
   </gazebo>
-  <gazebo reference="laser_base">
+  <gazebo reference="base_scan">
     <sensor type="ray" name="lidar">
       <pose>0 0 0 0 0 0</pose>
       <visualize>true</visualize>
-      <update_rate>40</update_rate>
+      <update_rate>50</update_rate>
       <ray>
         <scan>
@@ -458,11 +409,11 @@
             <samples>720</samples>
             <resolution>1</resolution>
-            <min_angle>-1.57</min_angle>
-            <max_angle>1.57</max_angle>
+            <min_angle>-1.57079</min_angle>
+            <max_angle>1.57079</max_angle>
           </horizontal>
         </scan>
         <range>
           <min>0.10</min>
-          <max>30.0</max>
+          <max>21.0</max>
           <resolution>0.01</resolution>
         </range>
@@ -479,12 +430,78 @@
       <plugin name="lidar_controller" filename="libgazebo_ros_laser.so">
         <!-- <robotNamespace>astrid</robotNamespace> -->
-        <topicName>astrid/scan</topicName>
-        <frameName>laser_base</frameName>
+        <topicName>scan</topicName>
+        <frameName>base_scan</frameName>
         <alwaysOn>true</alwaysOn>
       </plugin>
     </sensor>
   </gazebo>
+  <!-- Top View Camera-->
+  <joint name="top_view_camera_joint" type="fixed">
+    <axis xyz="0 1 0" />
+    <!-- <origin xyz="0 4.2 2.5" rpy="0 0.2 -1.57"/> -->
+    <origin xyz="-3 0 1.8" rpy="0 0 0" />
+    <parent link="shell"/>
+    <child link="top_view_camera_link"/>
+  </joint>
+  <link name="top_view_camera_link">
+    <visual>
+      <origin xyz="0 0 0" rpy="0 0 0"/>
+      <geometry>
+    <box size="0.05 0.07 0.03"/>
+      </geometry>
+      <material name="red"/>
+    </visual>
+    <inertial>
+      <mass value="1e-5" />
+      <origin xyz="0 0 0" rpy="0 0 0"/>
+      <inertia ixx="1e-6" ixy="0" ixz="0" iyy="1e-6" iyz="0" izz="1e-6" />
+    </inertial>
+  </link>
+<!-- top view camera -->
+    <gazebo reference="top_view_camera_link">
+      <sensor type="camera" name="top_view_camera">
+        <update_rate>30.0</update_rate>
+        <camera name="top_view_head">
+          <horizontal_fov>1.3962634</horizontal_fov>
+          <image>
+            <width>1600</width>
+            <height>900</height>
+            <format>R8G8B8</format>
+          </image>
+          <clip>
+            <near>0.02</near>
+            <far>500</far>
+          </clip>
+          <noise>
+            <type>gaussian</type>
+            <!-- Noise is sampled independently per pixel on each frame.
+                 That pixel's noise value is added to each of its color
+                 channels, which at that point lie in the range [0,1]. -->
+            <mean>0.0</mean>
+            <stddev>0.007</stddev>
+          </noise>
+        </camera>
+        <plugin name="camera_controller" filename="libgazebo_ros_camera.so">
+          <alwaysOn>true</alwaysOn>
+          <updateRate>0.0</updateRate>
+          <cameraName>astrid/top_view_camera</cameraName>
+          <imageTopicName>image_raw</imageTopicName>
+          <cameraInfoTopicName>camera_info</cameraInfoTopicName>
+          <frameName>camera_link</frameName>
+          <hackBaseline>0.07</hackBaseline>
+          <distortionK1>0.0</distortionK1>
+          <distortionK2>0.0</distortionK2>
+          <distortionK3>0.0</distortionK3>
+          <distortionT1>0.0</distortionT1>
+          <distortionT2>0.0</distortionT2>
+        </plugin>
+      </sensor>
+    </gazebo>
   <gazebo>
     <plugin name="gazebo_ros_control" filename="libgazebo_ros_control.so" />
+    <robotBaseFrame>base_link</robotBaseFrame>
+    <commandTopic>cmd_vel</commandTopic>
+      <odometryTopic>odom</odometryTopic>
+      <odometryFrame>odom</odometryFrame>
   </gazebo>
 </robot>
